File: hodiny.kicad_pcb (KiCad board)
At the start: 2 copper layers, 58 parts, among them U1 DS1302+, U10 4511, U11 4511, U12 4511, U2 4511, U8 4511, U9 4511, Y1 32.768kHz

Commit message: Add files via upload
Parts:
- added jumper 1: 0R, Resistor_THT:R_Axial_DIN0204_L3.6mm_D1.6mm_P5.08mm_Horizontal, F.Cu at (125.6, 84.0)
- added jumper 2: 0R, Resistor_THT:R_Axial_DIN0204_L3.6mm_D1.6mm_P5.08mm_Horizontal, F.Cu at (101.6, 84.5)
- A2, Y1: moved to B.Cu
- moved BT1 198.8 mm to (263.9, 138.5), turned to 180 degrees
- moved A2 186.0 mm to (234.6, 93.4), turned to -90 degrees
- moved U1 165.9 mm to (264.3, 114.7)
- moved Y1 151.5 mm to (260.9, 119.5), turned to 90 degrees
- moved R36 116.6 mm to (225.8, 95.5), turned to 180 degrees
- moved R41 112.2 mm to (225.6, 118.0), turned to 180 degrees
- moved R40 111.7 mm to (225.8, 109.0), turned to 180 degrees
- moved R39 111.5 mm to (225.8, 104.5), turned to 180 degrees
- moved R38 111.4 mm to (225.8, 100.0), turned to 180 degrees
- moved R37 111.3 mm to (225.8, 91.0), turned to 180 degrees
- moved R42 103.2 mm to (225.8, 113.5), turned to 180 degrees
- moved U12 103.0 mm to (206.1, 79.2), turned to 180 degrees
- moved DS10 95.2 mm to (190.1, 106.5)
- moved DS11 95.2 mm to (201.6, 106.5)
- moved U11 92.1 mm to (183.1, 79.2), turned to 180 degrees
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Routing:
- net +5V: track 0.00 -> 255.9 mm
- net Net-(A2-D4): track 0.00 -> 201.7 mm
- net Net-(A2-D6): track 0.00 -> 188.1 mm
- net Net-(A2-D3): track 0.00 -> 176.5 mm
- net Net-(A2-D7): track 0.00 -> 164.0 mm
- net Net-(A2-D8): track 0.00 -> 153.5 mm
- net Net-(A2-D5): track 0.00 -> 124.4 mm
- net Net-(A2-D2): track 0.00 -> 117.7 mm
- net Net-(A2-D9): track 0.00 -> 111.7 mm
- net Net-(A2-D10): track 0.00 -> 92.1 mm
- net Net-(U12-Qe): track 0.00 -> 87.6 mm
- net Net-(U12-Qd): track 0.00 -> 84.4 mm
- net Net-(A2-MOSI): track 0.00 -> 80.0 mm
- net Net-(U10-Qe): track 0.00 -> 78.5 mm
- net Net-(U10-Qd): track 0.00 -> 77.9 mm
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- added copper zone on B.Cu, net GND
- added copper zone on F.Cu, net GND
Other:
- board outline added: 250 x 96.5 mm

Commit message: Add files via upload
Parts:
- added J1: S1, Connector_PinHeader_2.54mm:PinHeader_1x02_P2.54mm_Horizontal, F.Cu at (138.3, 131.3)
- added J2: S2, Connector_PinHeader_2.54mm:PinHeader_1x02_P2.54mm_Horizontal, F.Cu at (138.3, 138.4)
- added J3: S3, Connector_PinHeader_2.54mm:PinHeader_1x02_P2.54mm_Horizontal, F.Cu at (138.3, 145.6)
Connections:
- A2 pad 22: unconnected-(A2-A3-Pad22) -> Net-(A2-A3)
- A2 pad 23: unconnected-(A2-SDA/A4-Pad23) -> Net-(A2-SDA/A4)
- A2 pad 24: unconnected-(A2-SCL/A5-Pad24) -> Net-(A2-SCL/A5)
Routing:
- net Net-(A2-D6): track 188.1 -> 193.2 mm
- net Net-(A2-D7): track 164.0 -> 169.1 mm
- net +5V: track 255.9 -> 258.4 mm
